Commit message: add app

File: cute_unit_description/urdf/cute_arm.urdf.xacro (robot description, xacro)
@@ -12,5 +12,5 @@
       <origin
         xyz="-0.00099787 0.019958 0.22081"
-        rpy="0 0 0" />
+        rpy="0 0 ${-PI/2}" />
       <mass
         value="9.0546" />
@@ -26,5 +26,5 @@
       <origin
         xyz="0 0 0"
-        rpy="0 0 0" />
+        rpy="0 0 ${-PI/2}" />
       <geometry>
         <mesh
@@ -48,5 +48,5 @@
       <origin
         xyz="0.0011123 -0.017941 0.13361"
-        rpy="0 0 0" />
+        rpy="0 0 ${PI}" />
       <mass
         value="9.0546" />
@@ -62,5 +62,5 @@
       <origin
         xyz="0 0 0"
-        rpy="0 0 0" />
+        rpy="0 0 ${PI}" />
       <geometry>
         <mesh
@@ -102,5 +102,5 @@
       <origin
         xyz="-0.00099787 0.018042 0.070815"
-        rpy="0 0 0" />
+        rpy="0 0 ${PI}" />
       <mass
         value="9.0546" />
@@ -116,5 +116,5 @@
       <origin
         xyz="0 0 0"
-        rpy="0 0 0" />
+        rpy="0 0 ${PI}" />
       <geometry>
         <mesh
@@ -156,5 +156,5 @@
       <origin
         xyz="-0.00099787 0.018033 -0.0060119"
-        rpy="0 0 0" />
+        rpy="0 0 ${PI}" />
       <mass
         value="9.0546" />
@@ -170,5 +170,5 @@
       <origin
         xyz="0 0 0"
-        rpy="0 0 0" />
+        rpy="0 0 ${PI}" />
       <geometry>
         <mesh
@@ -335,5 +335,5 @@
       <geometry>
         <mesh
-          filename="package://cute_model/meshes/cute_300es/part6.STL" />
+          filename="package://cute_model/meshes/cute_300es/part6_fix.STL" />
       </geometry>
       <material name="gray"/>
@@ -345,5 +345,5 @@
       <geometry>
         <mesh
-          filename="package://cute_model/meshes/cute_300es/part6.STL" />
+          filename="package://cute_model/meshes/cute_300es/part6_fix.STL" />
       </geometry>
     </collision>
@@ -354,5 +354,5 @@
     <origin
       xyz="0.00145 0 0.06663"
-      rpy="0 0 -1.8142" />
+      rpy="0 0 ${-PI/2}" />
     <parent
       link="part5" />
@@ -408,5 +408,5 @@
     <origin
       xyz="0 0 0.027"
-      rpy="0 0 -1.2645" />
+      rpy="0 0 ${-PI/2}" />
     <parent
       link="part6" />

File: cute_unit_description/urdf/cute_unit.urdf.xacro (robot description, xacro)
@@ -14,5 +14,5 @@
       </geometry>
       <material name="">
-        <color rgba="0.6 0.6 0.6 1" />
+        <color rgba="0.2 0.2 0.2 1.0" />
       </material>
     </visual>
@@ -27,5 +27,5 @@
   <cute_300es/>
   <joint name="arm_joint" type="fixed">
-    <origin xyz="-0.145 0 0.0335" rpy="0 0 -${M_PI/2}" />
+    <origin xyz="-0.145 0 0.0335" rpy="0 0 0" />
     <parent link="base_link"/>
     <child link="cute_base_link"/>
